File: 1bl.brd (EAGLE design)
At the start: 45.4 x 25.5 mm, 70 parts, among them IC1 78L05F, U1 ATMEGA168

Commit message: fw
Parts:
- C12: value (none) -> 10µF
- C9: value (none) -> 330µF/25V
- NA+, NB+, NC+: value IRFR5305 -> IRFR5305 oder FDD6637
- NA-, NB-, NC-: value IRFR5305 -> IRFR1205 oder IPD03N03LB oder IRLR7843
- R1, R12, R13, R18, R20, R21, R22, R4, R7: value (none) -> 4k7
- R10: value (none) -> 10K
- R11: value (none) -> 680R
- R14, R16, R23, R24: value (none) -> 18k
- R15: value (none) -> 1k
- R17, R19, R25: value (none) -> 100R
- R2, R5, R8: value (none) -> 470R
- R27, R33: value (none) -> 1K
- R3, R6, R9: value (none) -> 0R
- R32: value (none) -> 10R
- T1, T2, T3: value (none) -> PDTC143
